Commit message: sensor upgrade switching to rgbd camera

File: catkin_ws/src/my_robot/urdf/my_robot.xacro (robot description, xacro)
@@ -171,4 +171,6 @@
         </visual>
     </link>
+    <link name="camera_link_optical">
+    </link>
     <joint name="hokuyo_joint" type="fixed">
         <origin xyz="0.15 0 .1" rpy="0 0 0"/>
@@ -176,4 +178,9 @@
         <parent link="chassis"/>
         <child link="hokuyo"/>
+    </joint>
+    <joint name="camera_optical_joint" type="fixed">
+      <origin xyz="0 0 0" rpy="-1.5707 0 -1.5707"/>
+      <parent link="camera"/>
+      <child link="camera_link_optical"/>
     </joint>
     <gazebo reference="left_wheel">

Commit message: code cleaning and fixes robot camera

File: catkin_ws/src/my_robot/urdf/my_robot.xacro (robot description, xacro)
@@ -171,4 +171,9 @@
         </visual>
     </link>
+    <joint name="camera_optical_joint" type="fixed">
+      <origin xyz="0 0 0" rpy="-1.5707 0 -1.5707"/>
+      <parent link="camera"/>
+      <child link="camera_link_optical"/>
+    </joint>
     <link name="camera_link_optical">
     </link>
@@ -178,9 +183,4 @@
         <parent link="chassis"/>
         <child link="hokuyo"/>
-    </joint>
-    <joint name="camera_optical_joint" type="fixed">
-      <origin xyz="0 0 0" rpy="-1.5707 0 -1.5707"/>
-      <parent link="camera"/>
-      <child link="camera_link_optical"/>
     </joint>
     <gazebo reference="left_wheel">

Commit message: updating rviz config and other launch files

File: catkin_ws/src/my_robot/urdf/my_robot.xacro (robot description, xacro)
@@ -171,4 +171,6 @@
         </visual>
     </link>
+    <link name="camera_link_optical">
+    </link>
     <joint name="camera_optical_joint" type="fixed">
       <origin xyz="0 0 0" rpy="-1.5707 0 -1.5707"/>
@@ -176,6 +178,4 @@
       <child link="camera_link_optical"/>
     </joint>
-    <link name="camera_link_optical">
-    </link>
     <joint name="hokuyo_joint" type="fixed">
         <origin xyz="0.15 0 .1" rpy="0 0 0"/>
